Commit message: Update duckiebot model, add singleStreet world file, deleted useless world files

File: duckiebot_description/urdf/duckiebot.xacro (robot description, xacro)
@@ -36,5 +36,5 @@
       <origin xyz="0 0 0" rpy=" 0 0 0"/>
       <geometry>
-        <mesh filename="package://duckiebot_description/meshes/duckiebot_frame_only.dae"/>
+        <mesh filename="package://duckiebot_description/meshes/duckiebotFrame.dae"/>
       </geometry>
     </collision>
@@ -42,5 +42,5 @@
       <origin xyz="0 0 0" rpy=" 0 0 0"/>
       <geometry>
-        <mesh filename="package://duckiebot_description/meshes/duckiebot_frame_only.dae"/>
+        <mesh filename="package://duckiebot_description/meshes/duckiebotFrame.dae"/>
       </geometry>
       <material name="red"/>
@@ -67,7 +67,7 @@
       <cylinder_inertia m="${wheelMass}" r="0.0325" h="0.02"/>
       <inertia
-        ixx="1.56167e-05" ixy="0.0" ixz="0.0"
-        iyy="1.56167e-05" iyz="0.0"
-        izz="2.56e-05"/>
+        ixx="0.56167e-05" ixy="0.0" ixz="0.0"
+        iyy="0.56167e-05" iyz="0.0"
+        izz="1.56e-05"/>
     </inertial>
   </link>
@@ -92,7 +92,7 @@
       <cylinder_inertia m="${wheelMass}" r="0.0325" h="0.01"/>
       <inertia
-        ixx="1.56167e-05" ixy="0.0" ixz="0.0"
-        iyy="1.56167e-05" iyz="0.0"
-        izz="2.56e-05"/>
+        ixx="0.56167e-05" ixy="0.0" ixz="0.0"
+        iyy="0.56167e-05" iyz="0.0"
+        izz="1.56e-05"/>
     </inertial>
   </link>
